File: design/MeshRepeater2_Logic/Interconnect.kicad_sch (KiCad schematic)
At the start: 9 parts, among them J11 LC OUT - SYS 3V3, J201 INTERBOARD 12P

Commit message: Publish Mesh Repeater 2.0 A2
Add INA219 battery measurement with a 0.1 ohm shunt and vertical
12-pin interconnects through the middle shield. Publish updated
POWER, LOGIC and SHIELD KiCad sources, local models, BOM and A2
documentation with the completed routing and ground-via audit.

Preserve the V1 baseline and archives inside the V2 branch.
Validation: independent review 132/132; final artifact gate 499/499.
Parts:
- J201: value INTERBOARD 12P -> INTERBOARD 2x6 VERTICAL; footprint Meshcore:Connfly_DS1013_12RSIB_B_0_Horizontal__V2_J201 -> Meshcore:Ali_PinSocket_2x06_P2.54_H8.5_v2_mirror__V2_J201; MPN Connfly DS1013-12RSIB-B-0 -> MTJ H8.5 2X6P 10PCS; MPN_LTO_2S Connfly DS1013-12RSIB-B-0 -> MTJ H8.5 2X6P 10PCS; MPN_NaIon Connfly DS1013-12RSIB-B-0 -> MTJ H8.5 2X6P 10PCS; MPN_NaIon_NoCold Connfly DS1013-12RSIB-B-0 -> MTJ H8.5 2X6P 10PCS; Value_LTO_2S INTERBOARD 12P -> INTERBOARD 2x6 VERTICAL; Value_NaIon INTERBOARD 12P -> INTERBOARD 2x6 VERTICAL; Value_NaIon_NoCold INTERBOARD 12P -> INTERBOARD 2x6 VERTICAL; Vendor Danomsk -> AliExpress; Vendor URL https://www.danomsk.ru/shop/7-kommutatsiya/121-razemy/306-s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 -> https://aliexpress.ru/item/1005008954873458.html?sku_id=120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
Connections:
- net FILTER_OUT: no longer J201.7 (FILTER_OUT)
- net GND: no longer J201.10 (GND), J201.12 (GND)
- net SYS_3V3: now also J201.7 (SYS_3V3)
- new net SCL: J201.12 (SCL)
- new net SDA: J201.10 (SDA)
Other:
- note added: "MTJ H8.5 2X6P 10PCS"
- note added: "R21 оставлен 1 кОм: RADIO_TXEN → R21 → MODE через штыри."
- note added: "THT 2x6 / 2.54 / vertical"
- note added: "V2.0-A2 / 2026-10-12 / инженерный прототип"
- note added: "Распиновка прямого соединения — interboard_connections.csv."
- note removed: "DS1013-12RSIB-B-0"
- note removed: "IDC 2x6 / 2.54 / 90deg"
- note removed: "R21 оставлен 1 кОм: RADIO_TXEN → R21 → MODE через кабель."
- note removed: "V2.0-A1 / 2026-10-11 / инженерный прототип"
- note removed: "Полная распиновка и маршрут кабеля — interboard_connections.csv."
