File: design/MeshRepeater2_Logic/MeshRepeater2_Logic.kicad_pcb (KiCad board)
At the start: 2 copper layers, 90 x 60 mm, 57 parts, among them J10 AVR ISP 3V3, J11 LC OUT - SYS 3V3, J13 SMA 50Ohm, J201 INTERBOARD 12P, J3 I2C3V3, J4 GPS / T114 P3, J5 UART3V3, M1 NiceNano_CLONE_MODIFIED, M2 HT-RA62, Q2 AO3401A, Q3 2N7002K, SW1 USER, SW2 RESET, U4 DS3231MZ+TRL, U6 ATtiny13A-SSU, U7 SN74LVC2G125

Commit message: Publish Mesh Repeater 2.0 A2
Add INA219 battery measurement with a 0.1 ohm shunt and vertical
12-pin interconnects through the middle shield. Publish updated
POWER, LOGIC and SHIELD KiCad sources, local models, BOM and A2
documentation with the completed routing and ground-via audit.

Preserve the V1 baseline and archives inside the V2 branch.
Validation: independent review 132/132; final artifact gate 499/499.
Parts:
- J201: value INTERBOARD 12P -> INTERBOARD 2x6 VERTICAL; footprint Meshcore:Connfly_DS1013_12RSIB_B_0_Horizontal__V2_J201 -> Meshcore:Ali_PinSocket_2x06_P2.54_H8.5_v2_mirror__V2_J201
- moved J201 12.7 mm to (64.2, 49.0), turned to 90 degrees
Connections:
- J201 pad 10: GND -> SDA
- J201 pad 12: GND -> SCL
- J201 pad 7: FILTER_OUT -> SYS_3V3
Routing:
- net Net-(M2-MOSI): track 185.3 -> 30.9 mm, vias 11 -> 2
- net Net-(M1-P0.02_/_MISO): track 121.7 -> 42.5 mm, vias 11 -> 4
- net /RADIO_RST: track 105.1 -> 32.6 mm, vias 6 -> 1
- net SYS_3V3: track 322.9 -> 360.1 mm
- net SCL: track 107.4 -> 133.6 mm
- net SDA: track 102.1 -> 125.7 mm
- net /RADIO_RXEN: track 109.3 -> 96.1 mm, vias 5 -> 7
- net GND: track 55.9 -> 43.9 mm, vias 380 -> 423
- net FILTER_OUT: track 47.7 -> 59.0 mm, vias 0 -> 1
- net MODE: track 20.5 -> 29.6 mm
- net BAT: track 113.0 -> 118.1 mm
- net /RADIO_DIO1: track 32.8 -> 35.6 mm, vias 5 -> 7
- net Net-(M2-SCK): track 29.2 -> 30.0 mm, vias 2 -> 4
- net MCU_RESET: track 93.2 -> 92.7 mm
- net GPS_TX_MCU: track 82.1 -> 82.3 mm, vias 9 -> 11
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Other:
- board text added: "1/3/5 OUT | 2/4/6/8 GND"
- board text added: "11 MODE | 12 SCL"
- board text added: "7 3V3 | 9 BAT | 10 SDA"
- board text added: "J201 2x6 H8.5"
- board text removed: "1 3V3"
- board text removed: "10 GND"
- board text removed: "11 MODE"
- board text removed: "12 GND"
- board text removed: "3 3V3"
- board text removed: "4 GND"
- board text removed: "5 3V3"
- board text removed: "7 3V3"
- board text removed: "8 GND"
- board text removed: "9 BAT"
- board text removed: "J201"
- board text removed: "J201 IDC 12P"
