File: design/MeshRepeater2_Logic/MeshRepeater2_Logic.kicad_sch (KiCad schematic)
At the start: 22 parts, among them J13 SMA 50Ohm, M1 NiceNano_CLONE_MODIFIED, M2 HT-RA62, SW1 USER, SW2 RESET

Commit message: Publish Mesh Repeater 2.0 A2
Add INA219 battery measurement with a 0.1 ohm shunt and vertical
12-pin interconnects through the middle shield. Publish updated
POWER, LOGIC and SHIELD KiCad sources, local models, BOM and A2
documentation with the completed routing and ground-via audit.

Preserve the V1 baseline and archives inside the V2 branch.
Validation: independent review 132/132; final artifact gate 499/499.
Other:
- note added: "V2.0-A2 / 2026-10-12 / инженерный прототип"
- note removed: "V2.0-A1 / 2026-10-11 / инженерный прототип"
