File: design/MeshRepeater2_Logic/RTC_IO.kicad_sch (KiCad schematic)
At the start: 18 parts, among them J3 I2C3V3, J4 GPS / T114 P3, J5 UART3V3, Q2 AO3401A, Q3 2N7002K, U4 DS3231MZ+TRL, U7 SN74LVC2G125

Commit message: Publish Mesh Repeater 2.0 A2
Add INA219 battery measurement with a 0.1 ohm shunt and vertical
12-pin interconnects through the middle shield. Publish updated
POWER, LOGIC and SHIELD KiCad sources, local models, BOM and A2
documentation with the completed routing and ground-via audit.

Preserve the V1 baseline and archives inside the V2 branch.
Validation: independent review 132/132; final artifact gate 499/499.
Other:
- note added: "V2.0-A2 / 2026-10-12 / инженерный прототип"
- note removed: "V2.0-A1 / 2026-10-11 / инженерный прототип"
