File: design/MeshRepeater2_Logic/Watchdog.kicad_sch (KiCad schematic)
At the start: 8 parts, among them J10 AVR ISP 3V3, U6 ATtiny13A-SSU

Commit message: Publish Mesh Repeater 2.0 A2
Add INA219 battery measurement with a 0.1 ohm shunt and vertical
12-pin interconnects through the middle shield. Publish updated
POWER, LOGIC and SHIELD KiCad sources, local models, BOM and A2
documentation with the completed routing and ground-via audit.

Preserve the V1 baseline and archives inside the V2 branch.
Validation: independent review 132/132; final artifact gate 499/499.
Other:
- note added: "V2.0-A2 / 2026-10-12 / инженерный прототип"
- note removed: "V2.0-A1 / 2026-10-11 / инженерный прототип"
