File: design/MeshRepeater2_Power/Interconnect.kicad_sch (KiCad schematic)
At the start: 5 parts, among them J101 INTERBOARD 12P

Commit message: Publish Mesh Repeater 2.0 A2
Add INA219 battery measurement with a 0.1 ohm shunt and vertical
12-pin interconnects through the middle shield. Publish updated
POWER, LOGIC and SHIELD KiCad sources, local models, BOM and A2
documentation with the completed routing and ground-via audit.

Preserve the V1 baseline and archives inside the V2 branch.
Validation: independent review 132/132; final artifact gate 499/499.
Parts:
- H1, H2, H3, H4: Value_LTO_2S M3 NPTH -> M3 GND contact; Value_NaIon_NoCold M3 NPTH -> M3 GND contact
- J101: value INTERBOARD 12P -> INTERBOARD 2x6 VERTICAL; footprint Meshcore:Connfly_DS1013_12RSIB_B_0_Horizontal__V2_J101 -> Meshcore:Ali_PinHeader_2x06_P2.54_L35_A3C6__V2_J101; MPN Connfly DS1013-12RSIB-B-0 -> E-SIMPO L35mm A3C6 2x6P; MPN_LTO_2S Connfly DS1013-12RSIB-B-0 -> E-SIMPO L35mm A3C6 2x6P; MPN_NaIon Connfly DS1013-12RSIB-B-0 -> E-SIMPO L35mm A3C6 2x6P; MPN_NaIon_NoCold Connfly DS1013-12RSIB-B-0 -> E-SIMPO L35mm A3C6 2x6P; Value_LTO_2S INTERBOARD 12P -> INTERBOARD 2x6 VERTICAL; Value_NaIon INTERBOARD 12P -> INTERBOARD 2x6 VERTICAL; Value_NaIon_NoCold INTERBOARD 12P -> INTERBOARD 2x6 VERTICAL; Vendor Danomsk -> AliExpress; Vendor URL https://www.danomsk.ru/shop/7-kommutatsiya/121-razemy/306-s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 -> https://aliexpress.ru/item/1005011978353933.html?sku_id=120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
Connections:
- net FILTER_OUT: no longer J101.7 (FILTER_OUT)
- net GND: no longer J101.10 (GND), J101.12 (GND)
- new net SCL: J101.12 (SCL)
- new net SDA: J101.10 (SDA)
- new net SYS_3V3: J101.7 (SYS_3V3)
Other:
- note added: "E-SIMPO L35mm A3C6 2x6P"
- note added: "SYS_3V3 возвращается с LOGIC только для питания INA219."
- note added: "THT 2x6 / 2.54 / vertical"
- note added: "V2.0-A2 / 2026-10-12 / инженерный прототип"
- note added: "Основные токи FILTER_OUT и GND идут через вертикальные штыри."
- note added: "Распиновка прямого соединения — interboard_connections.csv."
- note removed: "DS1013-12RSIB-B-0"
- note removed: "IDC 2x6 / 2.54 / 90deg"
- note removed: "V2.0-A1 / 2026-10-11 / инженерный прототип"
- note removed: "Основные токи FILTER_OUT и GND идут по кабелю."
- note removed: "Полная распиновка и маршрут кабеля — interboard_connections.csv."
