File: design/MeshRepeater2_Power/MeshRepeater2_Power.kicad_pcb (KiCad board)
At the start: 2 copper layers, 90 x 60 mm, 115 parts, among them J101 INTERBOARD 12P, J12 LTO 2S + MID -, J7 SOLAR 12V, J8 Na-ion 1S, Q1 AO3401A, Q4 AO3401A, Q5 BSS138, Q6 AO3401A, Q7 AO3401A, U1 CN3722, U10 LM393XK, U11 LM285Z-2.5G, U2 TPS63802DLAR, U8 LMV431A, U9 LMV431A

Commit message: Publish Mesh Repeater 2.0 A2
Add INA219 battery measurement with a 0.1 ohm shunt and vertical
12-pin interconnects through the middle shield. Publish updated
POWER, LOGIC and SHIELD KiCad sources, local models, BOM and A2
documentation with the completed routing and ground-via audit.

Preserve the V1 baseline and archives inside the V2 branch.
Validation: independent review 132/132; final artifact gate 499/499.
Parts:
- added C63: 100nF 50V X7R, Meshcore:C_0805_2012Metric__V2_C63, B.Cu at (61.0, 11.4)
- added C64: 100nF 50V X7R, Meshcore:C_0805_2012Metric__V2_C64, B.Cu at (57.8, 7.70)
- added R71: 0.1R 1% 1W, Meshcore:R_2512_6332Metric__V2_R71, B.Cu at (46.5, 6.50)
- added R72: 10R 1%, Meshcore:R_0805_2012Metric__V2_R72, B.Cu at (54.0, 12.2)
- added R73: 10R 1%, Meshcore:R_0805_2012Metric__V2_R73, B.Cu at (54.0, 9.80)
- added U12: INA219AIDR, Meshcore:SOIC-8_3.9x4.9mm_P1.27mm__V2_U12, F.Cu at (58.2, 12.8)
- J101: value INTERBOARD 12P -> INTERBOARD 2x6 VERTICAL; footprint Meshcore:Connfly_DS1013_12RSIB_B_0_Horizontal__V2_J101 -> Meshcore:Ali_PinHeader_2x06_P2.54_L35_A3C6__V2_J101
Connections:
- C12 pad 1: BAT -> BAT_SYS
- C13 pad 1: BAT -> BAT_SYS
- C30 pad 1: BAT -> BAT_SYS
- C4 pad 1: BAT -> BAT_SYS
- C52 pad 1: BAT -> BAT_SYS
- C53 pad 1: BAT -> BAT_SYS
- J101 pad 10: GND -> SDA
- J101 pad 12: GND -> SCL
- J101 pad 7: FILTER_OUT -> SYS_3V3
- R1 pad 2: BAT -> BAT_SYS
- R3 pad 1: BAT -> BAT_SYS
- U1 pad 14: BAT -> BAT_SYS
- U2 pad 10: BAT -> BAT_SYS
Routing:
- net BAT_SYS: track 0.00 -> 91.7 mm, vias 0 -> 7
- net CHRG: track 99.3 -> 51.3 mm
- net SDA: track 0.00 -> 30.6 mm
- net SCL: track 0.00 -> 24.2 mm, vias 0 -> 1
- net BAT: track 230.3 -> 213.4 mm, vias 13 -> 9
- net FILTER_OUT: track 75.2 -> 58.9 mm
- net SYS_3V3: track 0.00 -> 13.8 mm, vias 0 -> 1
- net Net-(U12-IN-): track 0.00 -> 10.9 mm, vias 0 -> 1
- net GND: track 214.9 -> 208.9 mm, vias 482 -> 455
- net Net-(U12-IN+): track 0.00 -> 5.34 mm, vias 0 -> 2
- net LTO_MID: track 73.5 -> 70.6 mm
- net MODE: track 51.8 -> 50.0 mm
Other:
- board text added: "1 LC_OUT"
- board text added: "10 SDA"
- board text added: "12 SCL"
- board text added: "3 LC_OUT"
- board text added: "5 LC_OUT"
- board text added: "7 SYS_3V3"
- board text added: "C63 100nF"
- board text added: "C64"
- board text added: "C64 100nF"
- board text added: "D4"
- board text added: "G14 x1.5"
- board text added: "G3 x1.5"
- board text added: "G4 x2"
- board text added: "G6 x3"
- board text added: "J101 2x6 L35"
- board text added: "R71 0.1R"
- board text added: "R72 10R"
- board text added: "R73 10R"
- board text added: "U12"
- board text added: "U12 INA219AIDR"
- board text removed: "1 3V3"
- board text removed: "10 GND"
- board text removed: "12 GND"
- board text removed: "3 3V3"
- board text removed: "5 3V3"
- board text removed: "7 3V3"
- board text removed: "G3 x2"
- board text removed: "G4 x1.5"
- board text removed: "G6 x1.5"
- board text removed: "J101 IDC 12P"
- board text removed: "L3"
- board text removed: "R11"
