File: design/MeshRepeater2_Power/MeshRepeater2_Power.kicad_sch (KiCad schematic)
At the start: 30 parts, among them J7 SOLAR 12V, J8 Na-ion 1S, Q1 AO3401A, U1 CN3722

Commit message: Publish Mesh Repeater 2.0 A2
Add INA219 battery measurement with a 0.1 ohm shunt and vertical
12-pin interconnects through the middle shield. Publish updated
POWER, LOGIC and SHIELD KiCad sources, local models, BOM and A2
documentation with the completed routing and ground-via audit.

Preserve the V1 baseline and archives inside the V2 branch.
Validation: independent review 132/132; final artifact gate 499/499.
Parts:
- removed J8: Na-ion 1S, Meshcore:JST_XH_S2B-XH-A_1x02_P2.50mm_Horizontal__V2_J8, symbol Meshcore:J2
Connections:
- net BAT renamed BAT_SYS
Other:
- sheet 5. Interconnect renamed 6. Interconnect
- added sheet 5. BatteryMonitor (BatteryMonitor.kicad_sch)
- note added: "V2.0-A2 / 2026-10-12 / инженерный прототип"
- note removed: "V2.0-A1 / 2026-10-11 / инженерный прототип"
