File: design/Meshcore_NaIon/Converter.kicad_sch (KiCad schematic)
At the start: 45 parts, among them J11 LC OUT - SYS 3V3, U2 TPS63802DLAR

Commit message: Publish Mesh Repeater S4.16: routing fixes, COLD option and readable board labels
Update the editable KiCad project, seven-page schematic, portable footprints and 3D models, assembly variants, BOM, previews and independent CAD proofs. Preserve FakeTec GPIO compatibility. Manufacturing release remains paused.
Parts:
- added R55: 47mR 1%, Meshcore:R_Vishay_WSL1206_18, symbol Meshcore:R_H
- added TP8: FILTER_MID, Meshcore:TestPoint_Pad_D1.5mm, symbol Meshcore:TP
Connections:
- net FILTER_MID: now also TP8.1
- net SYS_PRE: now also R55.1; no longer L3.1
- new net SYS_LC_IN: L3.1, R55.2
Other:
- note added: "1206 / 0.25 W"
- note added: "FILTER_MID"
- note added: "R0470FEA"
- note added: "R55: 47 мОм последовательно перед L3; падение 47 мВ/А. FB и C14 до R55."
- note added: "S4.15 / 2026-10-11 / инженерный прототип"
- note added: "WSL1206"
- note removed: "S4.12 / 2026-10-10 / инженерный прототип"

Commit message: Publish S4.21 PCB and validated Rezonit manufacturing package
Update the public project to the accepted single-board S4.21 design, keeping
the user's manual routing improvements and removing SH1 and TP6.

Include the full editable KiCad project and local assets, three assembly BOM
variants, current assembly notes, eight-page schematic PDF, board views and
a clean nine-file Gerber/Excellon ZIP for Rezonit.

Validation: layout 29/29, power 14/14, CAM 59/59, publication integrity 18/18.
The committed native board and manufacturing ZIP match the verified byte
hashes. Preserve the existing licensing notices and watchdog source.
Parts:
- removed TP6: GND, Meshcore:TestPoint_Pad_D1.5mm, symbol Meshcore:TP
- added NT2: 3V3 STAR, Meshcore:NetTie_2_SMD_Power_Star_A3, symbol Meshcore:NETTIE
- C12, C52: Fit_NaIon_NoCold (none) -> yes; MPN_NaIon_NoCold (none) -> CL21B106KOQNNNE; Value_NaIon_NoCold (none) -> 10uF 16V X7R
- C13: Fit_NaIon_NoCold (none) -> yes; MPN_NaIon_NoCold (none) -> CL10B104KB8NNNC; Value_NaIon_NoCold (none) -> 100nF 50V X7R
- C14: Fit_NaIon_NoCold (none) -> yes; MPN_NaIon_NoCold (none) -> CL21A226MAQNNNE; Value_NaIon_NoCold (none) -> 22uF 25V X5R
- C15, C16, C34, C35, C36, C37, C38, C39, C40, C41, C42, C43, C44, C45, C46, C47, C48, C49, C50, C51: Fit_NaIon_NoCold (none) -> yes; MPN_NaIon_NoCold (none) -> C4532X5R1A107M280KC; Value_NaIon_NoCold (none) -> 100uF
- C53, C54, C55: Fit_NaIon_NoCold (none) -> no; Value_NaIon_NoCold (none) -> DNP
- J11: Fit_NaIon_NoCold (none) -> yes; MPN_NaIon_NoCold (none) -> DS1021-1X40SF11-B; Value_NaIon_NoCold (none) -> LC OUT - SYS 3V3
- L2: Fit_NaIon_NoCold (none) -> yes; MPN_NaIon_NoCold (none) -> XGL4020-471MEC; Value_NaIon_NoCold (none) -> 0.47uH
- L3, L4: Fit_NaIon_NoCold (none) -> yes; MPN_NaIon_NoCold (none) -> CDRH127/LDNP-2R4NC; Value_NaIon_NoCold (none) -> 2.4uH
- R13: Fit_NaIon_NoCold (none) -> yes; MPN_NaIon_NoCold (none) -> RNCF0805BKE56K0; Value_NaIon_NoCold (none) -> 56k 0.1%
- R14: Fit_NaIon_NoCold (none) -> yes; MPN_NaIon_NoCold (none) -> RT0805BRE0710KL; Value_NaIon_NoCold (none) -> 10k 0.1%
- R15: Fit_NaIon_NoCold (none) -> yes; MPN_NaIon_NoCold (none) -> RT0805BRD0740K2L; Value_NaIon_NoCold (none) -> 40.2k 0.1%
- R16: Fit_NaIon_NoCold (none) -> yes; MPN_NaIon_NoCold (none) -> RT0805BRD0749K9L; Value_NaIon_NoCold (none) -> 49.9k 0.1%
- R17: Fit_NaIon_NoCold (none) -> yes; MPN_NaIon_NoCold (none) -> RC0805FR-07100KL; Value_NaIon_NoCold (none) -> 100k
- R21: Fit_NaIon_NoCold (none) -> yes; MPN_NaIon_NoCold (none) -> RC0805FR-071KL; Value_NaIon_NoCold (none) -> 1k
- R40: footprint Meshcore:R_Vishay_WSL1206_18 -> Meshcore:R_Vishay_WSL2512_A3__A3_R40; Fit_NaIon_NoCold (none) -> yes; LCSC C4041551 -> (none); MPN WSL1206R0220FEA -> WSL2512R0220FEA; MPN_LTO_2S WSL1206R0220FEA -> WSL2512R0220FEA; MPN_NaIon WSL1206R0220FEA -> WSL2512R0220FEA; MPN_NaIon_NoCold (none) -> WSL2512R0220FEA; Package (none) -> 2512 / 1 W; Value_NaIon_NoCold (none) -> 22mR 1%
- R41: footprint Meshcore:R_Vishay_WSL1206_18 -> Meshcore:R_Vishay_WSL2512_A3__A3_R41; Fit_NaIon_NoCold (none) -> yes; LCSC C4041551 -> (none); MPN WSL1206R0220FEA -> WSL2512R0220FEA; MPN_LTO_2S WSL1206R0220FEA -> WSL2512R0220FEA; MPN_NaIon WSL1206R0220FEA -> WSL2512R0220FEA; MPN_NaIon_NoCold (none) -> WSL2512R0220FEA; Package (none) -> 2512 / 1 W; Value_NaIon_NoCold (none) -> 22mR 1%
- R55: footprint Meshcore:R_Vishay_WSL1206_18 -> Meshcore:R_Vishay_WSL2512_A3__A3_R55; Fit_NaIon_NoCold (none) -> yes; MPN WSL1206R0470FEA -> WSL2512R0470FEA; MPN_LTO_2S WSL1206R0470FEA -> WSL2512R0470FEA; MPN_NaIon WSL1206R0470FEA -> WSL2512R0470FEA; MPN_NaIon_NoCold (none) -> WSL2512R0470FEA; Package (none) -> 2512 / 1 W; Value_NaIon_NoCold (none) -> 47mR 1%; Vendor URL https://www.chipdip.ru/product/wsl1206r0470fea-current-sens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 -> (none)
- TP1: Fit_NaIon_NoCold (none) -> yes; Value_NaIon_NoCold (none) -> BAT
- TP3: Fit_NaIon_NoCold (none) -> yes; Value_NaIon_NoCold (none) -> SYS_PRE
- TP4: Fit_NaIon_NoCold (none) -> yes; Value_NaIon_NoCold (none) -> SYS_3V3
- TP7: Fit_NaIon_NoCold (none) -> yes; Value_NaIon_NoCold (none) -> GND
- TP8: Fit_NaIon_NoCold (none) -> yes; MPN_NaIon_NoCold (none) -> PCB test pad / not purchased; Value_NaIon_NoCold (none) -> FILTER_MID
- U2: Fit_NaIon_NoCold (none) -> yes; MPN_NaIon_NoCold (none) -> TPS63802DLAR; Value_NaIon_NoCold (none) -> TPS63802DLAR
Connections:
- net BAT: no longer C12.1, C13.1, C52.1, C53.1, U2.10 (VIN)
- net SYS_3V3: now also NT2.1
- new net BAT_SYS: C12.1, C13.1, C52.1, C53.1, U2.10 (VIN)
- new net RADIO_3V3: NT2.2
Other:
- note added: "2512 / 1 W"
- note added: "2: звезда SYS / RADIO"
- note added: "J11 → NT2: SYS_3V3 и отдельная RADIO_3V3. Снять ДО USB; вернуть после отключения USB."
- note added: "NT2: медная звезда, не разрезать"
- note added: "S4.17 / 2026-10-14 / инженерный прототип"
- note added: "WSL2512R0220FEA"
- note added: "WSL2512R0470FEA"
- note removed: "1206 / 0.25 W"
- note removed: "2: все нагрузки"
- note removed: "J11 соединяет выход LC с SYS_3V3 всех нагрузок. Снять ДО USB; вернуть после отключения USB."
- note removed: "R0470FEA"
- note removed: "S4.15 / 2026-10-11 / инженерный прототип"
- note removed: "WSL1206"
- note removed: "WSL1206, 1206 (3216)"
- note removed: "WSL1206R0220FEA"
