File: design/Meshcore_NaIon/LTO_Balancer.kicad_sch (KiCad schematic)
At the start: 13 parts, among them J12 LTO 2S + MID -, U8 LMV431A, U9 LMV431A

Commit message: Publish Mesh Repeater S4.16: routing fixes, COLD option and readable board labels
Update the editable KiCad project, seven-page schematic, portable footprints and 3D models, assembly variants, BOM, previews and independent CAD proofs. Preserve FakeTec GPIO compatibility. Manufacturing release remains paused.
Other:
- note added: "LTO: номинал 5,345 В; максимум 5,445 В при ТКС ≤25 ppm/°C, -40…85°C. Выбросы не учтены."
- note added: "Na-ion: R3=61,9k / R4=100k / C30=12pF. LTO: 121k / 100k / 6,8pF. Допуск R: 0,1%."
- note added: "S4.15 / 2026-10-11 / инженерный прототип"
- note added: "S4.15: отдельной защиты ячеек и защиты от перенапряжения нет."
- note removed: "LTO: номинал 5,408 В; угол до 5,481 В при ТКС ≤25 ppm/°C, -40…85°C. Выбросы не учтены."
- note removed: "Na-ion: R3=6,34k / R4=10k / C30=12pF. LTO: 13k / 10,5k / 6,8pF. Допуск R: 0,1%."
- note removed: "S4.12 / 2026-10-10 / инженерный прототип"
- note removed: "S4.12: отдельной защиты ячеек и защиты от перенапряжения нет."

Commit message: Publish S4.21 PCB and validated Rezonit manufacturing package
Update the public project to the accepted single-board S4.21 design, keeping
the user's manual routing improvements and removing SH1 and TP6.

Include the full editable KiCad project and local assets, three assembly BOM
variants, current assembly notes, eight-page schematic PDF, board views and
a clean nine-file Gerber/Excellon ZIP for Rezonit.

Validation: layout 29/29, power 14/14, CAM 59/59, publication integrity 18/18.
The committed native board and manufacturing ZIP match the verified byte
hashes. Preserve the existing licensing notices and watchdog source.
Parts:
- C58, C59: Fit_NaIon_NoCold (none) -> no; MPN_NaIon_NoCold (none) -> MPN TBD / 47nF X7R 16V; Value_NaIon_NoCold (none) -> 47nF 16V X7R
- J12: Fit_NaIon_NoCold (none) -> no; MPN_NaIon_NoCold (none) -> DS1021-1X40SF11-B; Value_NaIon_NoCold (none) -> LTO 2S + MID -
- R47, R51: Fit_NaIon_NoCold (none) -> no; MPN_NaIon_NoCold (none) -> RC0805FR-072RL; Value_NaIon_NoCold (none) -> 2R 1%
- R48, R52: Fit_NaIon_NoCold (none) -> no; MPN_NaIon_NoCold (none) -> MPN TBD / 120k 0.1%; Value_NaIon_NoCold (none) -> 120k 0.1%
- R49, R53: Fit_NaIon_NoCold (none) -> no; MPN_NaIon_NoCold (none) -> MPN TBD / 2.49k 0.1%; Value_NaIon_NoCold (none) -> 2.49k 0.1%
- R50, R54: Fit_NaIon_NoCold (none) -> no; MPN_NaIon_NoCold (none) -> MPN TBD / 100k 0.1%; Value_NaIon_NoCold (none) -> 100k 0.1%
- U8, U9: Fit_NaIon_NoCold (none) -> no; MPN_NaIon_NoCold (none) -> LMV431AIM5/NOPB; Value_NaIon_NoCold (none) -> LMV431A
Other:
- note added: "S4.17 / 2026-10-14 / инженерный прототип"
- note removed: "S4.15 / 2026-10-11 / инженерный прототип"
