File: design/Meshcore_NaIon/Modules.kicad_sch (KiCad schematic)
At the start: 19 parts, among them M1 NiceNano_CLONE_MODIFIED, M2 HT-RA62, SW1 USER, SW2 RESET

Commit message: Publish Mesh Repeater S4.16: routing fixes, COLD option and readable board labels
Update the editable KiCad project, seven-page schematic, portable footprints and 3D models, assembly variants, BOM, previews and independent CAD proofs. Preserve FakeTec GPIO compatibility. Manufacturing release remains paused.
Parts:
- added FL1: S869M000S003, Meshcore:SAW_AEL_DCC6C_S869M000S003, symbol Meshcore:SAW
- added J13: SMA 50Ohm, Meshcore:SMA_KLS1_SMA002_B_Horizontal, symbol Meshcore:COAX
- added NT1: Cu link / cut for FL1, Meshcore:RF_Cut_Link_0p6, symbol Meshcore:NETTIE
- R27, R28: value 1M 0.1% -> 2.2M 0.1%; MPN RT0805BRD071ML -> RG2012P-225-B-T5; MPN_LTO_2S RT0805BRD071ML -> RG2012P-225-B-T5; MPN_NaIon RT0805BRD071ML -> RG2012P-225-B-T5; Nominal 1M -> 2.2M; Value_LTO_2S 1M 0.1% -> 2.2M 0.1%; Value_NaIon 1M 0.1% -> 2.2M 0.1%; Vendor Danomsk -> ChipDip / Susumu; Vendor URL https://www.danomsk.ru/shop/6-rezistory/86-rezistory-postoy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 -> https://www.chipdip.ru/product/rg2012p-225-b-t5-susumu-8003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
Connections:
- net GND: now also FL1.1 (GND), FL1.3 (GND), FL1.4 (GND), FL1.6 (GND), J13.2 (SHIELD)
- net ANT_RF: now reaches M2.1 (ANT)
- net ANT_RF: now also FL1.2 (IN), NT1.1
- new net ANT_SMA: FL1.5 (OUT), J13.1 (RF), NT1.2
- no-connect marks 5 -> 4
Other:
- note added: "ADC: BAT/2; τ ≈ 110 мс. Калибровка ADC."
- note added: "DCC6C / 3 x 3 x 1.3 mm"
- note added: "FL1 — опция 868–870 МГц, TX ≤ +13 dBm. До установки разрезать медь NT1 под FL1. Без FL1 оставить NT1 целой."
- note added: "HT-RA62: R1 = 0 Ом (ANT); R2 снять (IPEX). R1/R2 здесь — резисторы внутри модуля. Подключать антенну только к J13."
- note added: "L-KLS1-SMA002-B"
- note added: "RG2012P-225-B-T5"
- note added: "S4.15 / 2026-10-11 / инженерный прототип"
- note added: "S869M000S003 / опция"
- note added: "SMA / угловой / PTH"
- note added: "SPI: 33 Ом у драйверов. ANT: J13 / SMA, 50 Ом. TXEN → MODE и watchdog. P1.06 свободен. BUSY=P0.29; GPS_EN=P0.24. GPS_EN=HIGH: питание GPS включено."
- note removed: "ADC: BAT/2; установление ≈ 50 мс."
- note removed: "RT0805BRD071ML"
- note removed: "S4.12 / 2026-10-10 / инженерный прототип"
- note removed: "SPI: 33 Ом у драйверов. ANT: штатный IPEX. TXEN → MODE и watchdog. P1.06 свободен. BUSY=P0.29; GPS_EN=P0.24. GPS_EN=HIGH: питание GPS включено."

Commit message: Publish S4.21 PCB and validated Rezonit manufacturing package
Update the public project to the accepted single-board S4.21 design, keeping
the user's manual routing improvements and removing SH1 and TP6.

Include the full editable KiCad project and local assets, three assembly BOM
variants, current assembly notes, eight-page schematic PDF, board views and
a clean nine-file Gerber/Excellon ZIP for Rezonit.

Validation: layout 29/29, power 14/14, CAM 59/59, publication integrity 18/18.
The committed native board and manufacturing ZIP match the verified byte
hashes. Preserve the existing licensing notices and watchdog source.
Parts:
- C21: Fit_NaIon_NoCold (none) -> yes; MPN_NaIon_NoCold (none) -> CL21B106KOQNNNE; Value_NaIon_NoCold (none) -> 10uF 16V X7R
- C22, C24, C25, C26: Fit_NaIon_NoCold (none) -> yes; MPN_NaIon_NoCold (none) -> CL21B104KBCNNNC; Value_NaIon_NoCold (none) -> 100nF 50V X7R
- C23: Fit_NaIon_NoCold (none) -> yes; MPN_NaIon_NoCold (none) -> CL21A226MAQNNNE; Value_NaIon_NoCold (none) -> 22uF 25V X5R
- FB1: Fit_NaIon_NoCold (none) -> yes; MPN_NaIon_NoCold (none) -> BLM21PG600SN1D; Value_NaIon_NoCold (none) -> 60R@100MHz / 3A
- FL1: Fit_NaIon_NoCold (none) -> no; MPN_NaIon_NoCold (none) -> S869M000S003; Value_NaIon_NoCold (none) -> S869M000S003
- J13: Fit_NaIon_NoCold (none) -> yes; MPN_NaIon_NoCold (none) -> L-KLS1-SMA002-B; Value_NaIon_NoCold (none) -> SMA 50Ohm
- M1: Fit_NaIon_NoCold (none) -> yes; MPN_NaIon_NoCold (none) -> User supplied NiceNano clone; Value_NaIon_NoCold (none) -> NiceNano_CLONE_MODIFIED
- M2: Fit_NaIon_NoCold (none) -> yes; MPN_NaIon_NoCold (none) -> HT-RA62 band variant TBD; Value_NaIon_NoCold (none) -> HT-RA62
- NT1: Fit_NaIon_NoCold (none) -> yes; MPN_NaIon_NoCold (none) -> PCB copper / not purchased; Value_NaIon_NoCold (none) -> Cu link / cut for FL1
- R23, R24, R25, R26: Fit_NaIon_NoCold (none) -> yes; MPN_NaIon_NoCold (none) -> RC0805FR-0733RL; Value_NaIon_NoCold (none) -> 33R
- R27, R28: Fit_NaIon_NoCold (none) -> yes; MPN_NaIon_NoCold (none) -> RG2012P-225-B-T5; Value_NaIon_NoCold (none) -> 2.2M 0.1%
- R31: Fit_NaIon_NoCold (none) -> yes; MPN_NaIon_NoCold (none) -> RC0805FR-0710KL; Value_NaIon_NoCold (none) -> 10k
- R35: Fit_NaIon_NoCold (none) -> yes; MPN_NaIon_NoCold (none) -> RC0805FR-07100KL; Value_NaIon_NoCold (none) -> 100k
- SW1: Fit_NaIon_NoCold (none) -> yes; MPN_NaIon_NoCold (none) -> KLS7-TS6604-4.3-180; Value_NaIon_NoCold (none) -> USER
- SW2: Fit_NaIon_NoCold (none) -> yes; MPN_NaIon_NoCold (none) -> KLS7-TS6604-4.3-180; Value_NaIon_NoCold (none) -> RESET
Connections:
- net RADIO_3V3: now also FB1.1; no longer C23.1, C24.1, FB1.2, M2.3 (3V3)
- net SYS_3V3: no longer FB1.1
- new net RADIO_LOCAL_3V3: C23.1, C24.1, FB1.2, M2.3 (3V3)
Other:
- note added: "NT2-звезда: SYS_3V3 → NiceNano / периферия; RADIO_3V3 → FB1 → RADIO_LOCAL_3V3."
- note added: "S4.17 / 2026-10-14 / инженерный прототип"
- note removed: "S4.15 / 2026-10-11 / инженерный прототип"
- note removed: "Модем: отдельная ветвь J11 → FB1 → RADIO_3V3. GPS/RTC питаются до FB1."
