File: design/Meshcore_NaIon/RTC_IO.kicad_sch (KiCad schematic)
At the start: 23 parts, among them J3 I2C3V3, J4 GPS / T114 P3, J5 UART3V3, Q2 AO3401A, Q3 2N7002K, U4 DS3231MZ+TRL, U7 SN74LVC2G125

Commit message: Publish Mesh Repeater S4.16: routing fixes, COLD option and readable board labels
Update the editable KiCad project, seven-page schematic, portable footprints and 3D models, assembly variants, BOM, previews and independent CAD proofs. Preserve FakeTec GPIO compatibility. Manufacturing release remains paused.
Other:
- note added: "S4.15 / 2026-10-11 / инженерный прототип"
- note removed: "S4.12 / 2026-10-10 / инженерный прототип"

Commit message: Publish S4.21 PCB and validated Rezonit manufacturing package
Update the public project to the accepted single-board S4.21 design, keeping
the user's manual routing improvements and removing SH1 and TP6.

Include the full editable KiCad project and local assets, three assembly BOM
variants, current assembly notes, eight-page schematic PDF, board views and
a clean nine-file Gerber/Excellon ZIP for Rezonit.

Validation: layout 29/29, power 14/14, CAM 59/59, publication integrity 18/18.
The committed native board and manufacturing ZIP match the verified byte
hashes. Preserve the existing licensing notices and watchdog source.
Parts:
- removed SH1: CUSTOM_SHIELD_FRAME, Meshcore:Shield_Frame_76x43, symbol Meshcore:J4
- BT1: Fit_NaIon_NoCold (none) -> yes; MPN_NaIon_NoCold (none) -> 1060; Value_NaIon_NoCold (none) -> CR2032 / holder
- C27, C56: Fit_NaIon_NoCold (none) -> yes; MPN_NaIon_NoCold (none) -> CL21B104KBCNNNC; Value_NaIon_NoCold (none) -> 100nF 50V X7R
- C57: Fit_NaIon_NoCold (none) -> yes; MPN_NaIon_NoCold (none) -> CL21B106KOQNNNE; Value_NaIon_NoCold (none) -> 10uF 16V X7R
- H1, H2, H3, H4: Fit_NaIon_NoCold (none) -> yes; Value_NaIon_NoCold (none) -> M3 NPTH
- J3: Fit_NaIon_NoCold (none) -> yes; MPN_NaIon_NoCold (none) -> DS1021-1X40SF11-B; Value_NaIon_NoCold (none) -> I2C3V3
- J4: Fit_NaIon_NoCold (none) -> yes; MPN_NaIon_NoCold (none) -> 53261-0871; Value_NaIon_NoCold (none) -> GPS / T114 P3
- J5: Fit_NaIon_NoCold (none) -> yes; MPN_NaIon_NoCold (none) -> DS1021-1X40SF11-B; Value_NaIon_NoCold (none) -> UART3V3
- Q2: Fit_NaIon_NoCold (none) -> yes; MPN_NaIon_NoCold (none) -> AO3401A; Value_NaIon_NoCold (none) -> AO3401A
- Q3: Fit_NaIon_NoCold (none) -> yes; MPN_NaIon_NoCold (none) -> 2N7002K; Value_NaIon_NoCold (none) -> 2N7002K
- R29, R30: Fit_NaIon_NoCold (none) -> yes; MPN_NaIon_NoCold (none) -> RC0805FR-074K7L; Value_NaIon_NoCold (none) -> 4.7k
- R42, R43, R45, R46: Fit_NaIon_NoCold (none) -> yes; MPN_NaIon_NoCold (none) -> RC0805FR-07100KL; Value_NaIon_NoCold (none) -> 100k
- R44: Fit_NaIon_NoCold (none) -> yes; MPN_NaIon_NoCold (none) -> RC0805FR-071KL; Value_NaIon_NoCold (none) -> 1k
- U4: Fit_NaIon_NoCold (none) -> yes; MPN_NaIon_NoCold (none) -> DS3231MZ+TRL; Value_NaIon_NoCold (none) -> DS3231MZ+TRL
- U7: Fit_NaIon_NoCold (none) -> yes; MPN_NaIon_NoCold (none) -> SN74LVC2G125DCTR; Value_NaIon_NoCold (none) -> SN74LVC2G125
Other:
- note added: "S4.17 / 2026-10-14 / инженерный прототип"
- note removed: "CUSTOM76x43x14mm"
- note removed: "S4.15 / 2026-10-11 / инженерный прототип"
- note removed: "custom frame76x43; H14"
- note removed: "Экран: внутренняя высота ≥ 14 мм; антенны снаружи."
