File: design/Meshcore_NaIon/Thermal.kicad_sch (KiCad schematic)
At the start: 24 parts, among them Q4 AO3401A, Q5 BSS138, Q6 AO3401A, Q7 AO3401A, U10 LM393XK, U11 LM285Z-2.5G

Commit message: Publish S4.21 PCB and validated Rezonit manufacturing package
Update the public project to the accepted single-board S4.21 design, keeping
the user's manual routing improvements and removing SH1 and TP6.

Include the full editable KiCad project and local assets, three assembly BOM
variants, current assembly notes, eight-page schematic PDF, board views and
a clean nine-file Gerber/Excellon ZIP for Rezonit.

Validation: layout 29/29, power 14/14, CAM 59/59, publication integrity 18/18.
The committed native board and manufacturing ZIP match the verified byte
hashes. Preserve the existing licensing notices and watchdog source.
Parts:
- C60, C62: Fit_NaIon_NoCold (none) -> no; MPN_NaIon_NoCold (none) -> CC0805KKX7R0BB104; Value_NaIon_NoCold (none) -> 100nF 100V X7R
- C61: Fit_NaIon_NoCold (none) -> no; MPN_NaIon_NoCold (none) -> CC0805JRNPO0BN102; Value_NaIon_NoCold (none) -> 1nF 100V C0G
- Q4, Q6, Q7: Fit_NaIon_NoCold (none) -> no; MPN_NaIon_NoCold (none) -> AO3401A; Value_NaIon_NoCold (none) -> AO3401A
- Q5: Fit_NaIon_NoCold (none) -> no; MPN_NaIon_NoCold (none) -> BSS138; Value_NaIon_NoCold (none) -> BSS138
- R57: Fit_NaIon_NoCold (none) -> no; MPN_NaIon_NoCold (none) -> RC0805FR-0747KL; Value_NaIon_NoCold (none) -> 47k 1% 0.125W
- R58, R59, R60, R61, R63: Fit_NaIon_NoCold (none) -> no; MPN_NaIon_NoCold (none) -> RC0805FR-07100KL; Value_NaIon_NoCold (none) -> 100k 1%
- R62, R67: Fit_NaIon_NoCold (none) -> no; MPN_NaIon_NoCold (none) -> RC0805FR-071ML; Value_NaIon_NoCold (none) -> 1M 1%
- R64: Fit_NaIon_NoCold (none) -> no; MPN_NaIon_NoCold (none) -> RC0805FR-071M2L; Value_NaIon_NoCold (none) -> 1.2M 1%
- R65: Fit_NaIon_NoCold (none) -> no; MPN_NaIon_NoCold (none) -> RC0805FR-0710KL; Value_NaIon_NoCold (none) -> 10k 1%
- R66, R68: Fit_NaIon_NoCold (none) -> no; MPN_NaIon_NoCold (none) -> RC0805FR-071KL; Value_NaIon_NoCold (none) -> 1k 1%
- R69: Fit_NaIon_NoCold (none) -> no; MPN_NaIon_NoCold (none) -> RC0805FR-0730KL; Value_NaIon_NoCold (none) -> 30k 1%
- R70: Fit_NaIon_NoCold (none) -> no; MPN_NaIon_NoCold (none) -> RC0805FR-07150KL; Value_NaIon_NoCold (none) -> 150k 1%
- TH1: Fit_NaIon_NoCold (none) -> no; MPN_NaIon_NoCold (none) -> B57861S0103F040; Value_NaIon_NoCold (none) -> 10k NTC 1% B3988
- U10: Fit_NaIon_NoCold (none) -> no; MPN_NaIon_NoCold (none) -> LM393XK; Value_NaIon_NoCold (none) -> LM393XK
- U11: Fit_NaIon_NoCold (none) -> no; MPN_NaIon_NoCold (none) -> LM285Z-2.5G; Value_NaIon_NoCold (none) -> LM285Z-2.5G
Other:
- note added: "S4.17 / 2026-10-14 / инженерный прототип"
- note removed: "S4.15 / 2026-10-11 / инженерный прототип"
