File: design/Meshcore_NaIon/Watchdog.kicad_sch (KiCad schematic)
At the start: 8 parts, among them J10 AVR ISP 3V3, U6 ATtiny13A-SSU

Commit message: Publish Mesh Repeater S4.16: routing fixes, COLD option and readable board labels
Update the editable KiCad project, seven-page schematic, portable footprints and 3D models, assembly variants, BOM, previews and independent CAD proofs. Preserve FakeTec GPIO compatibility. Manufacturing release remains paused.
Other:
- note added: "S4.15 / 2026-10-11 / инженерный прототип"
- note removed: "S4.12 / 2026-10-10 / инженерный прототип"

Commit message: Publish S4.21 PCB and validated Rezonit manufacturing package
Update the public project to the accepted single-board S4.21 design, keeping
the user's manual routing improvements and removing SH1 and TP6.

Include the full editable KiCad project and local assets, three assembly BOM
variants, current assembly notes, eight-page schematic PDF, board views and
a clean nine-file Gerber/Excellon ZIP for Rezonit.

Validation: layout 29/29, power 14/14, CAM 59/59, publication integrity 18/18.
The committed native board and manufacturing ZIP match the verified byte
hashes. Preserve the existing licensing notices and watchdog source.
Parts:
- C33: Fit_NaIon_NoCold (none) -> yes; MPN_NaIon_NoCold (none) -> CL21B104KBCNNNC; Value_NaIon_NoCold (none) -> 100nF 50V X7R
- J10: Fit_NaIon_NoCold (none) -> yes; MPN_NaIon_NoCold (none) -> DS1021-2X5SF11-B; Value_NaIon_NoCold (none) -> AVR ISP 3V3
- R33, R36: Fit_NaIon_NoCold (none) -> yes; MPN_NaIon_NoCold (none) -> RC0805FR-0710KL; Value_NaIon_NoCold (none) -> 10k
- R37: Fit_NaIon_NoCold (none) -> yes; MPN_NaIon_NoCold (none) -> RC0805FR-070RL; Value_NaIon_NoCold (none) -> 0R
- R38: Fit_NaIon_NoCold (none) -> yes; MPN_NaIon_NoCold (none) -> RC0805FR-071KL; Value_NaIon_NoCold (none) -> 1k
- R39: Fit_NaIon_NoCold (none) -> yes; MPN_NaIon_NoCold (none) -> RC0805FR-07100KL; Value_NaIon_NoCold (none) -> 100k
- U6: Fit_NaIon_NoCold (none) -> yes; MPN_NaIon_NoCold (none) -> ATTINY13A-SSU; Value_NaIon_NoCold (none) -> ATtiny13A-SSU
Other:
- note added: "S4.17 / 2026-10-14 / инженерный прототип"
- note removed: "S4.15 / 2026-10-11 / инженерный прототип"
